Commit message: Update urdf to have world-base link and turned upside down for move_gait.cpp

File: arm_description/urdf/arm.urdf (robot description, URDF)
Before this commit: robot arm, 5 links, 4 joints
Links:
- added link world
Joints:
- added joint base_joint: type fixed, parent world, child base, origin xyz=0 0 1.5 rpy=0 -3.14 0 
